Commit message: OpenAI Gym environnement

File: urdf_description/hexapod.urdf (robot description, URDF)
Before this commit: robot hexapod, 37 links, 36 joints
Links:
- link endcap_0: geometry collision sphere radius=0.005; visual sphere radius=0.005
- link endcap_1: geometry collision sphere radius=0.005; visual sphere radius=0.005
- link endcap_2: geometry collision sphere radius=0.005; visual sphere radius=0.005
- link endcap_3: geometry collision sphere radius=0.005; visual sphere radius=0.005
- link endcap_4: geometry collision sphere radius=0.005; visual sphere radius=0.005
- link endcap_5: geometry collision sphere radius=0.005; visual sphere radius=0.005
- link servomotor_0: geometry collision box size=0.024 .0451 .0347; visual box size=0.024 .0451 .0347
- link servomotor_1: geometry collision box size=0.024 .0451 .0347; visual box size=0.024 .0451 .0347
- link servomotor_10: geometry collision box size=0.024 .0451 .0347; visual box size=0.024 .0451 .0347
- link servomotor_11: geometry collision box size=0.024 .0451 .0347; visual box size=0.024 .0451 .0347
- link servomotor_12: geometry collision box size=0.024 .0451 .0347; visual box size=0.024 .0451 .0347
- link servomotor_13: geometry collision box size=0.024 .0451 .0347; visual box size=0.024 .0451 .0347
- link servomotor_14: geometry collision box size=0.024 .0451 .0347; visual box size=0.024 .0451 .0347
- link servomotor_15: geometry collision box size=0.024 .0451 .0347; visual box size=0.024 .0451 .0347
- link servomotor_16: geometry collision box size=0.024 .0451 .0347; visual box size=0.024 .0451 .0347
- link servomotor_17: geometry collision box size=0.024 .0451 .0347; visual box size=0.024 .0451 .0347
- link servomotor_2: geometry collision box size=0.024 .0451 .0347; visual box size=0.024 .0451 .0347
- link servomotor_3: geometry collision box size=0.024 .0451 .0347; visual box size=0.024 .0451 .0347
- link servomotor_4: geometry collision box size=0.024 .0451 .0347; visual box size=0.024 .0451 .0347
- link servomotor_5: geometry collision box size=0.024 .0451 .0347; visual box size=0.024 .0451 .0347
- link servomotor_6: geometry collision box size=0.024 .0451 .0347; visual box size=0.024 .0451 .0347
- link servomotor_7: geometry collision box size=0.024 .0451 .0347; visual box size=0.024 .0451 .0347
- link servomotor_8: geometry collision box size=0.024 .0451 .0347; visual box size=0.024 .0451 .0347
- link servomotor_9: geometry collision box size=0.024 .0451 .0347; visual box size=0.024 .0451 .0347
Joints:
- removed joint revolute_joint_0_servomotor_1
- removed joint revolute_joint_1_servomotor_4
- removed joint revolute_joint_2_servomotor_7
- removed joint revolute_joint_3_servomotor_10
- removed joint revolute_joint_4_servomotor_13
- removed joint revolute_joint_5_servomotor_16
- removed joint revolute_servomotor_0_joint_0
- removed joint revolute_servomotor_11_foot_3
- removed joint revolute_servomotor_12_joint_4
- removed joint revolute_servomotor_14_foot_4
- removed joint revolute_servomotor_15_joint_5
- removed joint revolute_servomotor_17_foot_5
- removed joint revolute_servomotor_2_foot_0
- removed joint revolute_servomotor_3_joint_1
- removed joint revolute_servomotor_5_foot_1
- removed joint revolute_servomotor_6_joint_2
- removed joint revolute_servomotor_8_foot_2
- removed joint revolute_servomotor_9_joint_3
- added joint servomotor_0: type revolute, parent servomotor_0, child joint_0, origin xyz=0 0.011 0 rpy=0 0 0, axis 0 0 1, limit lower=-1.57 upper=1.57 effort=1.18 velocity=6.308
- added joint servomotor_1: type revolute, parent joint_0, child servomotor_1, origin xyz=0.049 0 0 rpy=1.5707963267948966 -0.7853981633974483 0, axis 0 0 1, limit lower=-1.57 upper=1.57 effort=1.18 velocity=6.308
- added joint servomotor_10: type revolute, parent joint_3, child servomotor_10, origin xyz=0.049 0 0 rpy=1.5707963267948966 -0.7853981633974483 0, axis 0 0 1, limit lower=-1.57 upper=1.57 effort=1.18 velocity=6.308
- added joint servomotor_11: type revolute, parent servomotor_11, child foot_3, origin xyz=0 0.0107 0 rpy=0 0 -0.7853981633974483, axis 0 0 1, limit lower=-1.57 upper=1.57 effort=1.18 velocity=6.308
- added joint servomotor_12: type revolute, parent servomotor_12, child joint_4, origin xyz=0 0.011 0 rpy=0 0 3.141592653589793, axis 0 0 1, limit lower=-1.57 upper=1.57 effort=1.18 velocity=6.308
- added joint servomotor_13: type revolute, parent joint_4, child servomotor_13, origin xyz=0.049 0 0 rpy=1.5707963267948966 -0.7853981633974483 0, axis 0 0 1, limit lower=-1.57 upper=1.57 effort=1.18 velocity=6.308
- added joint servomotor_14: type revolute, parent servomotor_14, child foot_4, origin xyz=0 0.0107 0 rpy=0 0 -0.7853981633974483, axis 0 0 1, limit lower=-1.57 upper=1.57 effort=1.18 velocity=6.308
- added joint servomotor_15: type revolute, parent servomotor_15, child joint_5, origin xyz=0 0.011 0 rpy=0 0 3.141592653589793, axis 0 0 1, limit lower=-1.57 upper=1.57 effort=1.18 velocity=6.308
- added joint servomotor_16: type revolute, parent joint_5, child servomotor_16, origin xyz=0.049 0 0 rpy=1.5707963267948966 -0.7853981633974483 0, axis 0 0 1, limit lower=-1.57 upper=1.57 effort=1.18 velocity=6.308
- added joint servomotor_17: type revolute, parent servomotor_17, child foot_5, origin xyz=0 0.0107 0 rpy=0 0 -0.7853981633974483, axis 0 0 1, limit lower=-1.57 upper=1.57 effort=1.18 velocity=6.308
- added joint servomotor_2: type revolute, parent servomotor_2, child foot_0, origin xyz=0 0.0107 0 rpy=0 0 -0.7853981633974483, axis 0 0 1, limit lower=-1.57 upper=1.57 effort=1.18 velocity=6.308
- added joint servomotor_3: type revolute, parent servomotor_3, child joint_1, origin xyz=0 0.011 0 rpy=0 0 0, axis 0 0 1, limit lower=-1.57 upper=1.57 effort=1.18 velocity=6.308
- added joint servomotor_4: type revolute, parent joint_1, child servomotor_4, origin xyz=0.049 0 0 rpy=1.5707963267948966 -0.7853981633974483 0, axis 0 0 1, limit lower=-1.57 upper=1.57 effort=1.18 velocity=6.308
- added joint servomotor_5: type revolute, parent servomotor_5, child foot_1, origin xyz=0 0.0107 0 rpy=0 0 -0.7853981633974483, axis 0 0 1, limit lower=-1.57 upper=1.57 effort=1.18 velocity=6.308
- added joint servomotor_6: type revolute, parent servomotor_6, child joint_2, origin xyz=0 0.011 0 rpy=0 0 0, axis 0 0 1, limit lower=-1.57 upper=1.57 effort=1.18 velocity=6.308
- added joint servomotor_7: type revolute, parent joint_2, child servomotor_7, origin xyz=0.049 0 0 rpy=1.5707963267948966 -0.7853981633974483 0, axis 0 0 1, limit lower=-1.57 upper=1.57 effort=1.18 velocity=6.308
- added joint servomotor_8: type revolute, parent servomotor_8, child foot_2, origin xyz=0 0.0107 0 rpy=0 0 -0.7853981633974483, axis 0 0 1, limit lower=-1.57 upper=1.57 effort=1.18 velocity=6.308
- added joint servomotor_9: type revolute, parent servomotor_9, child joint_3, origin xyz=0 0.011 0 rpy=0 0 3.141592653589793, axis 0 0 1, limit lower=-1.57 upper=1.57 effort=1.18 velocity=6.308
- joint fixed_foot_0_endcap_0: origin xyz=0 0.0776 0 rpy=0 0 0 -> xyz=0 0.088 0 rpy=0 0 0
- joint fixed_foot_1_endcap_1: origin xyz=0 0.0776 0 rpy=0 0 0 -> xyz=0 0.088 0 rpy=0 0 0
- joint fixed_foot_2_endcap_2: origin xyz=0 0.0776 0 rpy=0 0 0 -> xyz=0 0.088 0 rpy=0 0 0
- joint fixed_foot_3_endcap_3: origin xyz=0 0.0776 0 rpy=0 0 0 -> xyz=0 0.088 0 rpy=0 0 0
- joint fixed_foot_4_endcap_4: origin xyz=0 0.0776 0 rpy=0 0 0 -> xyz=0 0.088 0 rpy=0 0 0
- joint fixed_foot_5_endcap_5: origin xyz=0 0.0776 0 rpy=0 0 0 -> xyz=0 0.088 0 rpy=0 0 0
