Commit message: Make OneLeg base static

File: gym_kraby/data/one_leg.urdf (robot description, URDF)
Before this commit: robot hexapod, 7 links, 6 joints
Joints:
- joint fixed_box_servomotor_0: origin xyz=0.06521292289492935 -0.06521292289492935 0.2041193 rpy=0 0 -0.78539 -> xyz=0.092225 0 0.2041193 rpy=0 0 0
