Commit message: Fix first servomotor collision

File: gym_kraby/data/hexapod.urdf (robot description, URDF)
Before this commit: robot hexapod, 37 links, 36 joints
Links:
- link foot_0: geometry collision box size=0.024 0.040 0.08; visual mesh filename=meshes/foot.stl scale=0.001 0.001 0.001
- link foot_1: geometry collision box size=0.024 0.040 0.08; visual mesh filename=meshes/foot.stl scale=0.001 0.001 0.001
- link foot_2: geometry collision box size=0.024 0.040 0.08; visual mesh filename=meshes/foot.stl scale=0.001 0.001 0.001
- link foot_3: geometry collision box size=0.024 0.040 0.08; visual mesh filename=meshes/foot.stl scale=0.001 0.001 0.001
- link foot_4: geometry collision box size=0.024 0.040 0.08; visual mesh filename=meshes/foot.stl scale=0.001 0.001 0.001
- link foot_5: geometry collision box size=0.024 0.040 0.08; visual mesh filename=meshes/foot.stl scale=0.001 0.001 0.001
- link joint_0: geometry collision box size=0.025 0.040 0.040; visual mesh filename=meshes/joint.stl scale=0.001 0.001 0.001
- link joint_1: geometry collision box size=0.025 0.040 0.040; visual mesh filename=meshes/joint.stl scale=0.001 0.001 0.001
- link joint_2: geometry collision box size=0.025 0.040 0.040; visual mesh filename=meshes/joint.stl scale=0.001 0.001 0.001
- link joint_3: geometry collision box size=0.025 0.040 0.040; visual mesh filename=meshes/joint.stl scale=0.001 0.001 0.001
- link joint_4: geometry collision box size=0.025 0.040 0.040; visual mesh filename=meshes/joint.stl scale=0.001 0.001 0.001
- link joint_5: geometry collision box size=0.025 0.040 0.040; visual mesh filename=meshes/joint.stl scale=0.001 0.001 0.001
- link servomotor_0: geometry collision box size=0.024 0.0451 0.0347; visual box size=0.024 0.0451 0.0347
- link servomotor_1: geometry collision box size=0.024 0.0451 0.0347; visual box size=0.024 0.0451 0.0347
- link servomotor_10: geometry collision box size=0.024 0.0451 0.0347; visual box size=0.024 0.0451 0.0347
- link servomotor_11: geometry collision box size=0.024 0.0451 0.0347; visual box size=0.024 0.0451 0.0347
- link servomotor_12: geometry collision box size=0.024 0.0451 0.0347; visual box size=0.024 0.0451 0.0347
- link servomotor_13: geometry collision box size=0.024 0.0451 0.0347; visual box size=0.024 0.0451 0.0347
- link servomotor_14: geometry collision box size=0.024 0.0451 0.0347; visual box size=0.024 0.0451 0.0347
- link servomotor_15: geometry collision box size=0.024 0.0451 0.0347; visual box size=0.024 0.0451 0.0347
- link servomotor_16: geometry collision box size=0.024 0.0451 0.0347; visual box size=0.024 0.0451 0.0347
- link servomotor_17: geometry collision box size=0.024 0.0451 0.0347; visual box size=0.024 0.0451 0.0347
- link servomotor_2: geometry collision box size=0.024 0.0451 0.0347; visual box size=0.024 0.0451 0.0347
- link servomotor_3: geometry collision box size=0.024 0.0451 0.0347; visual box size=0.024 0.0451 0.0347
- link servomotor_4: geometry collision box size=0.024 0.0451 0.0347; visual box size=0.024 0.0451 0.0347
- link servomotor_5: geometry collision box size=0.024 0.0451 0.0347; visual box size=0.024 0.0451 0.0347
- link servomotor_6: geometry collision box size=0.024 0.0451 0.0347; visual box size=0.024 0.0451 0.0347
- link servomotor_7: geometry collision box size=0.024 0.0451 0.0347; visual box size=0.024 0.0451 0.0347
- link servomotor_8: geometry collision box size=0.024 0.0451 0.0347; visual box size=0.024 0.0451 0.0347
- link servomotor_9: geometry collision box size=0.024 0.0451 0.0347; visual box size=0.024 0.0451 0.0347
Joints:
- joint servomotor_0: limit lower=-1.57 upper=1.57 effort=1.18 velocity=6.308 -> lower=-0.46 upper=0.46 effort=1.18 velocity=6.308
- joint servomotor_12: limit lower=-1.57 upper=1.57 effort=1.18 velocity=6.308 -> lower=-0.46 upper=0.46 effort=1.18 velocity=6.308
- joint servomotor_15: limit lower=-1.57 upper=1.57 effort=1.18 velocity=6.308 -> lower=-0.46 upper=0.46 effort=1.18 velocity=6.308
- joint servomotor_3: limit lower=-1.57 upper=1.57 effort=1.18 velocity=6.308 -> lower=-0.46 upper=0.46 effort=1.18 velocity=6.308
- joint servomotor_6: limit lower=-1.57 upper=1.57 effort=1.18 velocity=6.308 -> lower=-0.46 upper=0.46 effort=1.18 velocity=6.308
- joint servomotor_9: limit lower=-1.57 upper=1.57 effort=1.18 velocity=6.308 -> lower=-0.46 upper=0.46 effort=1.18 velocity=6.308

File: gym_kraby/data/one_leg.urdf (robot description, URDF)
Before this commit: robot hexapod, 7 links, 6 joints
Links:
- link foot_0: geometry collision box size=0.024 0.040 0.08; visual mesh filename=meshes/foot.stl scale=0.001 0.001 0.001
- link joint_0: geometry collision box size=0.025 0.040 0.040; visual mesh filename=meshes/joint.stl scale=0.001 0.001 0.001
- link servomotor_0: geometry collision box size=0.024 0.0451 0.0347; visual box size=0.024 0.0451 0.0347
- link servomotor_1: geometry collision box size=0.024 0.0451 0.0347; visual box size=0.024 0.0451 0.0347
- link servomotor_2: geometry collision box size=0.024 0.0451 0.0347; visual box size=0.024 0.0451 0.0347
Joints:
- joint servomotor_0: limit lower=-1.57 upper=1.57 effort=1.18 velocity=6.308 -> lower=-0.46 upper=0.46 effort=1.18 velocity=6.308
